File: STM32F401RE lite board.kicad_sch (KiCad schematic)
At the start: 25 parts, among them J1 USB_B_Micro, J2 Conn_01x04_Pin, SW1 SW_Push, SW2 SW_SPDT, Y1 8MHz(16pF)

Commit message: C1
Parts:
- removed J2: Conn_01x04_Pin, symbol Connector:Conn_01x04_Pin
- added C13, C16: 1µF_X5R, symbol Device:C
- added C14, C17: 100nF, symbol Device:C
- added C15: 10nF_X7R, symbol Device:C
- added D1: BAT60A, Diode_SMD:D_SOD-323, symbol Diode:BAT60A
- added J3: Conn_01x05_Pin, symbol Connector:Conn_01x05_Pin
- added U1: USBLC6-2SC6, Package_TO_SOT_SMD:SOT-23-6, symbol Power_Protection:USBLC6-2SC6
- added U2: LD3985M33R_SOT23, Package_TO_SOT_SMD:SOT-23-5, symbol Regulator_Linear:LD3985M33R_SOT23
- gave numbers to parts that had none: 1
Connections:
- net +3.3V: now also C16.1, C17.1, J3.1 (Pin_1), U2.5 (VOUT)
- net GND: now also C13.2, C14.2, C15.2, C16.2, C17.2, J3.5 (Pin_5), U1.2 (GND), U2.2 (GND)
- net NRST: now also J3.4 (Pin_4)
- net SWCLK: now also J3.3 (Pin_3)
- net SWDIO: now also J3.2 (Pin_2)
- net VBUS: now also D1.2 (A), U1.5 (VBUS)
- net at R6.1: now also U1.6 (I/O1); no longer J1.3 (D+)
- net at J1.2 (D-): now also U1.3 (I/O2); no longer R5.1
- new net: C13.1, C14.1, D1.1 (K), U2.1 (VIN), U2.3 (INH)
- new net: C15.1, U2.4 (BYP)
- new net: J1.3 (D+), U1.1 (I/O1)
- new net: R5.1, U1.4 (I/O2)
Other:
- note added: "MCU & USB"
- note added: "POWER SUPPLY"
- moved on the sheet: C1, C10, C11, C12, C2, C3, C4, C5, C6, C7, C8, C9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

Commit message: C2
Parts:
- added C18: 4.7µF, symbol Device:C
- added D2: LED, symbol Device:LED
- added J2, J4: Conn_01x04_Pin, symbol Connector:Conn_01x04_Pin
- added J5: Conn_01x05_Pin, symbol Connector:Conn_01x05_Pin
- added R7: 1KΩ, symbol Device:R
Connections:
- net +3.3V: now also D2.2 (A), J2.1 (Pin_1), J4.1 (Pin_1), J5.1 (Pin_1)
- net GND: now also C18.2, J2.4 (Pin_4), J4.4 (Pin_4), J5.5 (Pin_5), R7.2
- net PA5/SPI_SCK: now reaches U3.21 (PA5)
- net PA5/SPI_SCK: now also J5.2 (Pin_2)
- net PA6/SPI_MISO: now reaches U3.22 (PA6)
- net PA6/SPI_MISO: now also J5.3 (Pin_3)
- net PA7/SPI_MOSI: now reaches U3.23 (PA7)
- net PA7/SPI_MOSI: now also J5.4 (Pin_4)
- net at U3.30 (VCAP1): now also C18.1
- net PA9/UART_TX: now reaches U3.42 (PA9)
- net PA9/UART_TX: now also J4.2 (Pin_2)
- net PA10/UART_RX: now reaches U3.43 (PA10)
- net PA10/UART_RX: now also J4.3 (Pin_3)
- net PB6/I2C_SCL: now reaches U3.58 (PB6)
- net PB6/I2C_SCL: now also J2.2 (Pin_2)
- net PB7/I2C_SDA: now reaches U3.59 (PB7)
- net PB7/I2C_SDA: now also J2.3 (Pin_3)
- new net PWR_LED K: D2.1 (K), R7.1
Other:
- note added: "I2C CONNECTORS"
- note added: "SPI CONNECTORS"
- note added: "UART CONNECTORS"
- moved on the sheet: C1, C10, C11, C12, C13, C14, C15, C16, C17, C2, C3, C4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

Commit message: C3
Parts:
- added D3: LED, symbol Device:LED
- added J7: Conn_01x19_Pin, symbol Connector:Conn_01x19_Pin
- added J8: Conn_01x22_Pin, symbol Connector:Conn_01x22_Pin
- added R10, R9: 4.7KΩ, symbol Device:R
- added R8: 1KΩ, symbol Device:R
Connections:
- net +3.3V: now also J8.1 (Pin_1), R10.1, R9.1
- net GND: now also J7.2 (Pin_2), J8.2 (Pin_2), R8.2
- net PB6/I2C_SCL: now also R10.2
- net PB7/I2C_SDA: now also R9.2
- net VBUS: now also J7.1 (Pin_1)
- net PC2: now reaches U3.10 (PC2)
- net PC2: now also J7.6 (Pin_6)
- net PC3: now reaches U3.11 (PC3)
- net PC3: now also J7.7 (Pin_7)
- net PA0: now reaches U3.14 (PA0)
- net PA0: now also J8.3 (Pin_3)
- net PA1: now reaches U3.15 (PA1)
- net PA1: now also J8.4 (Pin_4)
- net PA2: now reaches U3.16 (PA2)
- net PA2: now also J8.5 (Pin_5)
- net PA3: now reaches U3.17 (PA3)
- net PA3: now also J8.6 (Pin_6)
- net PC13: now reaches U3.2 (PC13)
- net PC13: now also J7.17 (Pin_17)
- net PA4: now reaches U3.20 (PA4)
- net PA4: now also J8.7 (Pin_7)
- net PC4: now reaches U3.24 (PC4)
- net PC4: now also J7.8 (Pin_8)
- net PC5: now reaches U3.25 (PC5)
- net PC5: now also J7.9 (Pin_9)
- net PB0: now reaches U3.26 (PB0)
- net PB0: now also D3.2 (A), J8.10 (Pin_10)
- net PB1: now reaches U3.27 (PB1)
- net PB1: now also J8.11 (Pin_11)
- net PB2: now reaches U3.28 (PB2)
- net PB2: now also J8.12 (Pin_12)
- net PB10: now reaches U3.29 (PB10)
- net PB10: now also J8.18 (Pin_18)
- net PC14: now reaches U3.3 (PC14)
- net PC14: now also J7.18 (Pin_18)
- net PB12: now reaches U3.33 (PB12)
- net PB12: now also J8.19 (Pin_19)
- net PB13: now reaches U3.34 (PB13)
- net PB13: now also J8.20 (Pin_20)
- net PB14: now reaches U3.35 (PB14)
- net PB14: now also J8.21 (Pin_21)
- net PB15: now reaches U3.36 (PB15)
- net PB15: now also J8.22 (Pin_22)
- net PC6: now reaches U3.37 (PC6)
- net PC6: now also J7.10 (Pin_10)
- net PC7: now reaches U3.38 (PC7)
- net PC7: now also J7.11 (Pin_11)
- net PC8: now reaches U3.39 (PC8)
- net PC8: now also J7.12 (Pin_12)
- net PC15: now reaches U3.4 (PC15)
- net PC15: now also J7.19 (Pin_19)
- net PC9: now reaches U3.40 (PC9)
- net PC9: now also J7.13 (Pin_13)
- net PA8: now reaches U3.41 (PA8)
- net PA8: now also J8.8 (Pin_8)
- net PA15: now reaches U3.50 (PA15)
- net PA15: now also J8.9 (Pin_9)
- net PC10: now reaches U3.51 (PC10)
- net PC10: now also J7.14 (Pin_14)
- net PC11: now reaches U3.52 (PC11)
- net PC11: now also J7.15 (Pin_15)
- net PC12: now reaches U3.53 (PC12)
- net PC12: now also J7.16 (Pin_16)
- net PD2: now reaches U3.54 (PD2)
- net PD2: now also J7.3 (Pin_3)
- net PB3: now reaches U3.55 (PB3)
- net PB3: now also J8.13 (Pin_13)
- net PB4: now reaches U3.56 (PB4)
- net PB4: now also J8.14 (Pin_14)
- net PB5: now reaches U3.57 (PB5)
- net PB5: now also J8.15 (Pin_15)
- net PB8: now reaches U3.61 (PB8)
- net PB8: now also J8.16 (Pin_16)
- net PB9: now reaches U3.62 (PB9)
- net PB9: now also J8.17 (Pin_17)
- net PC0: now reaches U3.8 (PC0)
- net PC0: now also J7.4 (Pin_4)
- net PC1: now reaches U3.9 (PC1)
- net PC1: now also J7.5 (Pin_5)
- new net USER_LED_K: D3.1 (K), R8.1
Other:
- note added: "GPIO EXPANSIONS"
- moved on the sheet: C18

Commit message: C4
Parts:
- C1, C10, C11, C12, C13, C15, C16, C17, C2, C3, C4, C7, C8: footprint (none) -> Capacitor_SMD:C_0402_1005Metric
- C14, C18, C5, C6, C9: footprint (none) -> Capacitor_SMD:C_0603_1608Metric
- D2, D3: footprint (none) -> LED_SMD:LED_0603_1608Metric
- FB1: footprint (none) -> Inductor_SMD:L_0603_1608Metric
- J1: footprint (none) -> Connector_USB:USB_Micro-B_Molex-105017-0001
- Y1: footprint (none) -> Crystal:Crystal_SMD_HC49-SD
Changed lines of the file:
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@@
 	(text "POWER SUPPLY"
 		(exclude_from_sim no)
-		(at 22.86 15.24 0)
+		(at 30.48 16.51 0)
 		(effects
 			(font
-				(size 1.5 1.5)
+				(size 2.5 2.5)
 				(thickness 0.3)
 				(bold yes)
@@
 	(text "MCU & USB"
 		(exclude_from_sim no)
-		(at 116.84 15.24 0)
+		(at 122.682 16.764 0)
 		(effects
 			(font
-				(size 1.5 1.5)
+				(size 2.5 2.5)
 				(thickness 0.3)
 				(bold yes)
@@
 	(text "UART CONNECTORS\n"
 		(exclude_from_sim no)
-		(at 121.92 149.86 0)
+		(at 125.476 148.844 0)
 		(effects
 			(font
@@
 			)
 		)
-		(property "Footprint" ""
+		(property "Footprint" "Capacitor_SMD:C_0402_1005Metric"
 			(at 31.4452 40.64 0)
 			(effects
@@
 			)
 		)
-		(property "Footprint" ""
+		(property "Footprint" "Capacitor_SMD:C_0402_1005Metric"
 			(at 82.2452 40.64 0)
 			(effects
@@
 			)
 		)
-		(property "Footprint" ""
+		(property "Footprint" "LED_SMD:LED_0603_1608Metric"
 			(at 87.63 27.94 0)
 			(effects
@@
 			)
 		)
-		(property "Footprint" ""
+		(property "Footprint" "Capacitor_SMD:C_0402_1005Metric"
 			(at 145.7452 35.56 0)
 			(effects
@@
 			)
 		)
-		(property "Footprint" ""
+		(property "Footprint" "Capacitor_SMD:C_0603_1608Metric"
 			(at 152.4 44.7548 0)
 			(effects
@@
 			)
 		)
-		(property "Footprint" ""
+		(property "Footprint" "Capacitor_SMD:C_0402_1005Metric"
 			(at 135.5852 35.56 0)
 			(effects
@@
 			)
 		)
-		(property "Footprint" ""
+		(property "Footprint" "Crystal:Crystal_SMD_HC49-SD"
 			(at 134.62 105.41 0)
 			(effects
@@
 			)
 		)
-		(property "Footprint" ""
+		(property "Footprint" "Capacitor_SMD:C_0402_1005Metric"
 			(at 69.5452 40.64 0)
 			(effects
@@
 			)
 		)
-		(property "Footprint" ""
+		(property "Footprint" "Connector_USB:USB_Micro-B_Molex-105017-0001"
 			(at 245.11 72.39 0)
 			(effects
@@
 			)
 		)
-		(property "Footprint" ""
+		(property "Footprint" "Capacitor_SMD:C_0402_1005Metric"
 			(at 153.3652 63.5 0)
 			(effects
@@
 			)
 		)
-		(property "Footprint" ""
+		(property "Footprint" "Capacitor_SMD:C_0603_1608Metric"
 			(at 163.5252 124.46 0)
 			(effects
@@
 			)
 		)
-		(property "Footprint" ""
+		(property "Footprint" "Capacitor_SMD:C_0402_1005Metric"
 			(at 129.54 98.0948 0)
 			(effects
@@
 			)
 		)
-		(property "Footprint" ""
+		(property "Footprint" "Inductor_SMD:L_0603_1608Metric"
 			(at 130.81 55.118 90)
 			(effects
@@
 			)
 		)
-		(property "Footprint" ""
+		(property "Footprint" "Capacitor_SMD:C_0402_1005Metric"
 			(at 168.6052 35.56 0)
 			(effects
@@
 			)
 		)
-		(property "Footprint" ""
+		(property "Footprint" "Capacitor_SMD:C_0402_1005Metric"
 			(at 275.2852 66.04 0)
 			(effects
@@
 			)
 		)
-		(property "Footprint" ""
+		(property "Footprint" "LED_SMD:LED_0603_1608Metric"
 			(at 41.91 185.42 0)
 			(effects
@@
 			)
 		)
-		(property "Footprint" ""
+		(property "Footprint" "Capacitor_SMD:C_0402_1005Metric"
 			(at 158.4452 35.56 0)
 			(effects
@@
 			)
 		)
-		(property "Footprint" ""
+		(property "Footprint" "Capacitor_SMD:C_0402_1005Metric"
 			(at 59.3852 40.64 0)
 			(effects
@@
 			)
 		)
-		(property "Footprint" ""
+		(property "Footprint" "Capacitor_SMD:C_0402_1005Metric"
 			(at 129.54 108.2548 0)
 			(effects
@@
 			)
 		)
-		(property "Footprint" ""
+		(property "Footprint" "Capacitor_SMD:C_0603_1608Metric"
 			(at 122.8852 35.56 0)
 			(effects
@@
 			)
 		)
-		(property "Footprint" ""
+		(property "Footprint" "Capacitor_SMD:C_0603_1608Metric"
 			(at 140.6652 63.5 0)
 			(effects
@@
 			)
 		)
-		(property "Footprint" ""
+		(property "Footprint" "Capacitor_SMD:C_0402_1005Metric"
 			(at 120.3452 63.5 0)
 			(effects
@@
 			)
 		)
-		(property "Footprint" ""
+		(property "Footprint" "Capacitor_SMD:C_0603_1608Metric"
 			(at 39.0652 40.64 0)
 			(effects

Commit message: C5
Parts:
- J2, J4: footprint (none) -> Connector_PinHeader_2.54mm:PinHeader_1x04_P2.54mm_Vertical
- J3, J5: footprint (none) -> Connector_PinHeader_2.54mm:PinHeader_1x05_P2.54mm_Vertical
- J7: footprint (none) -> Connector_PinHeader_2.54mm:PinHeader_1x19_P2.54mm_Vertical
- J8: footprint (none) -> Connector_PinHeader_2.54mm:PinHeader_1x22_P2.54mm_Vertical
- R1, R10, R2, R3, R4, R5, R6, R7, R8, R9: footprint (none) -> Resistor_SMD:R_0402_1005Metric
- SW1: footprint (none) -> Button_Switch_SMD:SW_Push_1TS009xxxx-xxxx-xxxx_6x6x5mm
- SW2: footprint (none) -> Button_Switch_SMD:SW_SPST_B3U-1000P
- Y1: footprint Crystal:Crystal_SMD_HC49-SD -> Crystal:Crystal_HC49-4H_Vertical
Changed lines of the file:
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@@
 			)
 		)
-		(property "Footprint" ""
+		(property "Footprint" "Connector_PinHeader_2.54mm:PinHeader_1x04_P2.54mm_Vertical"
 			(at 63.5 76.2 0)
 			(effects
@@
 			)
 		)
-		(property "Footprint" ""
+		(property "Footprint" "Resistor_SMD:R_0402_1005Metric"
 			(at 222.25 71.882 90)
 			(effects
@@
 			)
 		)
-		(property "Footprint" ""
+		(property "Footprint" "Connector_PinHeader_2.54mm:PinHeader_1x22_P2.54mm_Vertical"
 			(at 58.42 147.32 0)
 			(effects
@@
 			)
 		)
-		(property "Footprint" ""
+		(property "Footprint" "Connector_PinHeader_2.54mm:PinHeader_1x04_P2.54mm_Vertical"
 			(at 124.46 160.02 0)
 			(effects
@@
 			)
 		)
-		(property "Footprint" ""
+		(property "Footprint" "Connector_PinHeader_2.54mm:PinHeader_1x19_P2.54mm_Vertical"
 			(at 40.64 144.78 0)
 			(effects
@@
 			)
 		)
-		(property "Footprint" "Crystal:Crystal_SMD_HC49-SD"
+		(property "Footprint" "Crystal:Crystal_HC49-4H_Vertical"
 			(at 134.62 105.41 0)
 			(effects
@@
 			)
 		)
-		(property "Footprint" ""
+		(property "Footprint" "Connector_PinHeader_2.54mm:PinHeader_1x05_P2.54mm_Vertical"
 			(at 30.48 76.2 0)
 			(effects
@@
 			)
 		)
-		(property "Footprint" ""
+		(property "Footprint" "Resistor_SMD:R_0402_1005Metric"
 			(at 92.202 36.83 90)
 			(effects
@@
 			)
 		)
-		(property "Footprint" ""
+		(property "Footprint" "Resistor_SMD:R_0402_1005Metric"
 			(at 265.938 64.77 90)
 			(effects
@@
 			)
 		)
-		(property "Footprint" ""
+		(property "Footprint" "Button_Switch_SMD:SW_Push_1TS009xxxx-xxxx-xxxx_6x6x5mm"
 			(at 157.48 35.56 0)
 			(effects
@@
 			)
 		)
-		(property "Footprint" ""
+		(property "Footprint" "Resistor_SMD:R_0402_1005Metric"
 			(at 54.61 187.198 90)
 			(effects
@@
 			)
 		)
-		(property "Footprint" ""
+		(property "Footprint" "Connector_PinHeader_2.54mm:PinHeader_1x05_P2.54mm_Vertical"
 			(at 134.62 185.42 0)
 			(effects
@@
 			)
 		)
-		(property "Footprint" ""
+		(property "Footprint" "Resistor_SMD:R_0402_1005Metric"
 			(at 222.25 69.342 90)
 			(effects
@@
 			)
 		)
-		(property "Footprint" ""
+		(property "Footprint" "Resistor_SMD:R_0402_1005Metric"
 			(at 79.502 67.31 90)
 			(effects
@@
 			)
 		)
-		(property "Footprint" ""
+		(property "Footprint" "Button_Switch_SMD:SW_SPST_B3U-1000P"
 			(at 129.54 83.82 0)
 			(effects
@@
 			)
 		)
-		(property "Footprint" ""
+		(property "Footprint" "Resistor_SMD:R_0402_1005Metric"
 			(at 138.43 85.598 90)
 			(effects
@@
 			)
 		)
-		(property "Footprint" ""
+		(property "Footprint" "Resistor_SMD:R_0402_1005Metric"
 			(at 146.05 100.838 90)
 			(effects
@@
 			)
 		)
-		(property "Footprint" ""
+		(property "Footprint" "Resistor_SMD:R_0402_1005Metric"
 			(at 74.422 66.04 90)
 			(effects
@@
 			)
 		)
-		(property "Footprint" ""
+		(property "Footprint" "Resistor_SMD:R_0402_1005Metric"
 			(at 146.05 110.998 90)
 			(effects

Commit message: C6
Parts:
- SW2: footprint Button_Switch_SMD:SW_SPST_B3U-1000P -> Button_Switch_SMD:SW_SPDT_CK_JS102011SAQN
Changed lines of the file:
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@@
 			)
 		)
-		(property "Footprint" "Button_Switch_SMD:SW_SPST_B3U-1000P"
+		(property "Footprint" "Button_Switch_SMD:SW_SPDT_CK_JS102011SAQN"
 			(at 129.54 83.82 0)
 			(effects

Commit message: C7
Parts:
- C18, C5, C6: footprint Capacitor_SMD:C_0603_1608Metric -> Capacitor_SMD:C_0805_2012Metric
Changed lines of the file:
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@@
 	)
 	(junction
-		(at 35.56 27.94)
-		(diameter 0)
-		(color 0 0 0 0)
-	)
-	(junction
 		(at 187.96 132.08)
 		(diameter 0)
@@
 	)
 	(junction
+		(at 35.56 27.94)
+		(diameter 0)
+		(color 0 0 0 0)
+	)
+	(junction
 		(at 68.58 43.18)
 		(diameter 0)
@@
 	(wire
 		(pts
-			(xy 35.56 27.94) (xy 38.1 27.94)
-		)
-		(stroke
-			(width 0)
-			(type default)
-		)
-	)
-	(wire
-		(pts
 			(xy 205.74 73.66) (xy 218.44 73.66)
 		)
@@
 	(wire
 		(pts
+			(xy 35.56 22.86) (xy 35.56 27.94)
+		)
+		(stroke
+			(width 0)
+			(type default)
+		)
+	)
+	(wire
+		(pts
 			(xy 170.18 43.18) (xy 165.1 43.18)
 		)
@@
 	(wire
 		(pts
+			(xy 35.56 27.94) (xy 38.1 27.94)
+		)
+		(stroke
+			(width 0)
+			(type default)
+		)
+	)
+	(wire
+		(pts
 			(xy 139.7 185.42) (xy 142.24 185.42)
 		)
@@
 	(symbol
 		(lib_id "power:PWR_FLAG")
-		(at 35.56 27.94 0)
+		(at 35.56 22.86 0)
 		(unit 1)
 		(exclude_from_sim no)
@@
 		(on_board yes)
 		(dnp no)
-		(fields_autoplaced yes)
 		(property "Reference" "#FLG02"
-			(at 35.56 26.035 0)
+			(at 35.56 20.955 0)
 			(effects
 				(font
@@
 		)
 		(property "Value" "PWR_FLAG"
-			(at 35.56 23.622 0)
+			(at 35.56 18.542 0)
 			(effects
 				(font
@@
 		)
 		(property "Footprint" ""
-			(at 35.56 27.94 0)
+			(at 35.56 22.86 0)
 			(effects
 				(font
@@
 		)
 		(property "Datasheet" "~"
-			(at 35.56 27.94 0)
+			(at 35.56 22.86 0)
 			(effects
 				(font
@@
 		)
 		(property "Description" "Special symbol for telling ERC where power comes from"
-			(at 35.56 27.94 0)
+			(at 35.56 22.86 0)
 			(effects
 				(font
@@
 			)
 		)
-		(property "Footprint" "Capacitor_SMD:C_0603_1608Metric"
+		(property "Footprint" "Capacitor_SMD:C_0805_2012Metric"
 			(at 163.5252 124.46 0)
 			(effects
@@
 			)
 		)
-		(property "Footprint" "Capacitor_SMD:C_0603_1608Metric"
+		(property "Footprint" "Capacitor_SMD:C_0805_2012Metric"
 			(at 122.8852 35.56 0)
 			(effects
@@
 			)
 		)
-		(property "Footprint" "Capacitor_SMD:C_0603_1608Metric"
+		(property "Footprint" "Capacitor_SMD:C_0805_2012Metric"
 			(at 140.6652 63.5 0)
 			(effects

Commit message: C9
Parts:
- removed R5, R6: 22Ω, Resistor_SMD:R_0402_1005Metric, symbol Device:R
- removed U1: USBLC6-2SC6, Package_TO_SOT_SMD:SOT-23-6, symbol Power_Protection:USBLC6-2SC6
Connections:
- net D +: now also J1.3 (D+)
- net D -: now also J1.2 (D-)
Other:
- moved on the sheet: C12, R4
