File: STM32F401RE lite board.kicad_sch (KiCad schematic)
At the start: 42 parts, among them J1 USB_B_Micro, J2 Conn_01x04_Pin, J3 Conn_01x05_Pin, J4 Conn_01x04_Pin, J5 Conn_01x05_Pin, J7 Conn_01x19_Pin, J8 Conn_01x22_Pin, SW1 SW_Push, SW2 SW_SPDT, U2 LD3985M33R_SOT23, U3 STM32F401RETx, Y1 8MHz(16pF)

Commit message: C10
Parts:
- removed J1: USB_B_Micro, Connector_USB:USB_Micro-B_Molex-105017-0001, symbol Connector:USB_B_Micro
- removed J2, J4: Conn_01x04_Pin, Connector_PinHeader_2.54mm:PinHeader_1x04_P2.54mm_Vertical, symbol Connector:Conn_01x04_Pin
- removed J5: Conn_01x05_Pin, Connector_PinHeader_2.54mm:PinHeader_1x05_P2.54mm_Vertical, symbol Connector:Conn_01x05_Pin
- removed J7: Conn_01x19_Pin, Connector_PinHeader_2.54mm:PinHeader_1x19_P2.54mm_Vertical, symbol Connector:Conn_01x19_Pin
- removed J8: Conn_01x22_Pin, Connector_PinHeader_2.54mm:PinHeader_1x22_P2.54mm_Vertical, symbol Connector:Conn_01x22_Pin
- removed R10, R9: 4.7KΩ, Resistor_SMD:R_0402_1005Metric, symbol Device:R
- removed SW1: SW_Push, Button_Switch_SMD:SW_Push_1TS009xxxx-xxxx-xxxx_6x6x5mm, symbol Switch:SW_Push
- removed SW2: SW_SPDT, Button_Switch_SMD:SW_SPDT_CK_JS102011SAQN, symbol Switch:SW_SPDT
- added J2: USB_C_Receptacle_USB2.0_16P, Connector_USB:USB_C_Receptacle_HRO_TYPE-C-31-M-12, symbol Connector:USB_C_Receptacle_USB2.0_16P
- added J6, J9: Conn_01x24_Pin, Connector_PinHeader_2.54mm:PinHeader_1x24_P2.54mm_Vertical, symbol Connector:Conn_01x24_Pin
- added R5, R6: 4.7KΩ, Resistor_SMD:R_0402_1005Metric, symbol Device:R
- added SW3, SW4: SW_SPST, Button_Switch_SMD:SW_SPST_TL3342, symbol Switch:SW_SPST
- R1: value 10KΩ -> 5.1KΩ
- R2: value 0Ω -> 10KΩ
- R3: value 0Ω -> 5.1KΩ
Connections:
- net +3.3V: now also J9.1 (Pin_1), R5.1, R6.1, SW3.2 (B)
- net BOOT0: now also R2.2, SW3.1 (A); no longer R1.2
- net D +: now also J2.A6 (D+), J2.B6 (D+)
- net D -: now also J2.A7 (D-), J2.B7 (D-)
- net GND: now also R1.2, R2.1, R3.1, J2.A1 (GND), J2.A12 (GND), J2.B1 (GND), J2.B12 (GND), J9.2 (Pin_2), SW4.2 (B)
- net NRST: now also SW4.1 (A)
- net OSC_IN: now also C10.2, Y1.2; no longer R3.2
- net OSC_OUT: now also C11.2, Y1.1; no longer R2.2
- net PA0: now also J6.23 (Pin_23)
- net PA1: now also J6.24 (Pin_24)
- net PA10/UART_RX: now also J6.2 (Pin_2)
- net PA15: now also J6.4 (Pin_4)
- net PA2: now also J9.24 (Pin_24)
- net PA3: now also J9.23 (Pin_23)
- net PA4: now also J9.22 (Pin_22)
- net PA5/SPI_SCK: now also J9.21 (Pin_21)
- net PA6/SPI_MISO: now also J9.20 (Pin_20)
- net PA7/SPI_MOSI: now also J9.19 (Pin_19)
- net PA8: now also J9.3 (Pin_3)
- net PA9/UART_TX: now also J6.3 (Pin_3)
- net PB0: now also J9.16 (Pin_16)
- net PB1: now also J9.15 (Pin_15)
- net PB10: now also J9.13 (Pin_13)
- net PB12: now also J9.12 (Pin_12)
- net PB13: now also J9.11 (Pin_11)
- net PB14: now also J9.10 (Pin_10)
- net PB15: now also J9.9 (Pin_9)
- net PB2: now also J9.14 (Pin_14)
- net PB3: now also J6.9 (Pin_9)
- net PB4: now also J6.10 (Pin_10)
- net PB5: now also J6.11 (Pin_11)
- net PB6/I2C_SCL: now also J6.12 (Pin_12), R5.2
- net PB7/I2C_SDA: now also J6.13 (Pin_13), R6.2
- net PB8: now also J6.14 (Pin_14)
- net PB9: now also J6.15 (Pin_15)
- net PC0: now also J6.19 (Pin_19)
- net PC1: now also J6.20 (Pin_20)
- net PC10: now also J6.5 (Pin_5)
- net PC11: now also J6.6 (Pin_6)
- net PC12: now also J6.7 (Pin_7)
- net PC13: now also J6.16 (Pin_16)
- net PC14: now also J6.17 (Pin_17)
- net PC15: now also J6.18 (Pin_18)
- net PC2: now also J6.21 (Pin_21)
- net PC3: now also J6.22 (Pin_22)
- net PC4: now also J9.18 (Pin_18)
- net PC5: now also J9.17 (Pin_17)
- net PC6: now also J9.8 (Pin_8)
- net PC7: now also J9.7 (Pin_7)
- net PC8: now also J9.5 (Pin_5), J9.6 (Pin_6)
- net PC9: now also J9.4 (Pin_4)
- net PD2: now also J6.8 (Pin_8)
- net VBUS: now also J2.A4 (VBUS), J2.A9 (VBUS), J2.B4 (VBUS), J2.B9 (VBUS), J6.1 (Pin_1)
- net at C12.1, R4.2: now also J2.S1 (SHIELD)
- net at R1.1: now also J2.A5 (CC1)
- new net: J2.B5 (CC2), R3.2
- no-connect marks 1 -> 2
Other:
- note removed: "I2C CONNECTORS"
- note removed: "SPI CONNECTORS"
- note removed: "UART CONNECTORS"
- moved on the sheet: C1, C10, C11, C12, C14, C18, C2, C3, C4, C5, C6, C7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

Commit message: C12
Connections:
- net +3.3V: now also J6.1 (Pin_1); no longer J9.1 (Pin_1)
- net GND: now also J6.2 (Pin_2)
- net PA0: now also J9.22 (Pin_22); no longer J6.23 (Pin_23)
- net PA1: now also J9.23 (Pin_23); no longer J6.24 (Pin_24)
- net PA10/UART_RX: now also J6.3 (Pin_3); no longer J6.2 (Pin_2)
- net PA15: now also J9.3 (Pin_3); no longer J6.4 (Pin_4)
- net PA3: now also J6.24 (Pin_24); no longer J9.23 (Pin_23)
- net PA4: now also J6.23 (Pin_23); no longer J9.22 (Pin_22)
- net PA5/SPI_SCK: now also J6.22 (Pin_22); no longer J9.21 (Pin_21)
- net PA6/SPI_MISO: now also J6.21 (Pin_21); no longer J9.20 (Pin_20)
- net PA7/SPI_MOSI: now also J6.20 (Pin_20); no longer J9.19 (Pin_19)
- net PA8: now also J6.5 (Pin_5); no longer J9.3 (Pin_3)
- net PA9/UART_TX: now also J6.4 (Pin_4); no longer J6.3 (Pin_3)
- net PB0: now also J6.17 (Pin_17); no longer J9.16 (Pin_16)
- net PB1: now also J6.16 (Pin_16); no longer J9.15 (Pin_15)
- net PB10: now also J6.14 (Pin_14); no longer J9.13 (Pin_13)
- net PB12: now also J6.13 (Pin_13); no longer J9.12 (Pin_12)
- net PB13: now also J6.12 (Pin_12); no longer J9.11 (Pin_11)
- net PB14: now also J6.11 (Pin_11); no longer J9.10 (Pin_10)
- net PB15: now also J6.10 (Pin_10); no longer J9.9 (Pin_9)
- net PB2: now also J6.15 (Pin_15); no longer J9.14 (Pin_14)
- net PB3: now also J9.8 (Pin_8); no longer J6.9 (Pin_9)
- net PB4: now also J9.9 (Pin_9); no longer J6.10 (Pin_10)
- net PB5: now also J9.10 (Pin_10); no longer J6.11 (Pin_11)
- net PB6/I2C_SCL: now also J9.11 (Pin_11); no longer J6.12 (Pin_12)
- net PB7/I2C_SDA: now also J9.12 (Pin_12); no longer J6.13 (Pin_13)
- net PB8: now also J9.13 (Pin_13); no longer J6.14 (Pin_14)
- net PB9: now also J9.14 (Pin_14); no longer J6.15 (Pin_15)
- net PC0: now also J9.18 (Pin_18); no longer J6.19 (Pin_19)
- net PC1: now also J9.19 (Pin_19); no longer J6.20 (Pin_20)
- net PC10: now also J9.4 (Pin_4); no longer J6.5 (Pin_5)
- net PC11: now also J9.5 (Pin_5); no longer J6.6 (Pin_6)
- net PC12: now also J9.6 (Pin_6); no longer J6.7 (Pin_7)
- net PC13: now also J9.15 (Pin_15); no longer J6.16 (Pin_16)
- net PC14: now also J9.16 (Pin_16); no longer J6.17 (Pin_17)
- net PC15: now also J9.17 (Pin_17); no longer J6.18 (Pin_18)
- net PC2: now also J9.20 (Pin_20); no longer J6.21 (Pin_21)
- net PC3: now also J9.21 (Pin_21); no longer J6.22 (Pin_22)
- net PC4: now also J6.19 (Pin_19); no longer J9.18 (Pin_18)
- net PC5: now also J6.18 (Pin_18); no longer J9.17 (Pin_17)
- net PC6: now also J6.9 (Pin_9); no longer J9.8 (Pin_8)
- net PC7: now also J6.8 (Pin_8); no longer J9.7 (Pin_7)
- net PC8: now also J6.7 (Pin_7); no longer J9.5 (Pin_5), J9.6 (Pin_6)
- net PC9: now also J6.6 (Pin_6); no longer J9.4 (Pin_4)
- net PD2: now also J9.7 (Pin_7); no longer J6.8 (Pin_8)
- net VBUS: now also J9.1 (Pin_1); no longer J6.1 (Pin_1)

Commit message: C14
Connections:
- net +3.3V: now also J9.1 (Pin_1); no longer J6.1 (Pin_1)
- net VBUS: now also J6.1 (Pin_1); no longer J9.1 (Pin_1)
Changed lines of the file:
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@@
 	(symbol
 		(lib_id "power:VBUS")
-		(at 63.5 109.22 270)
-		(unit 1)
-		(exclude_from_sim no)
-		(in_bom yes)
-		(on_board yes)
-		(dnp no)
-		(fields_autoplaced yes)
+		(at 30.48 109.22 270)
+		(unit 1)
+		(exclude_from_sim no)
+		(in_bom yes)
+		(on_board yes)
+		(dnp no)
 		(property "Reference" "#PWR035"
-			(at 59.69 109.22 0)
+			(at 26.67 109.22 0)
 			(effects
 				(font
@@
 		)
 		(property "Value" "VBUS"
-			(at 68.834 109.2199 90)
+			(at 34.29 109.22 90)
 			(effects
 				(font
@@
 		)
 		(property "Footprint" ""
-			(at 63.5 109.22 0)
+			(at 30.48 109.22 0)
 			(effects
 				(font
@@
 		)
 		(property "Datasheet" ""
-			(at 63.5 109.22 0)
+			(at 30.48 109.22 0)
 			(effects
 				(font
@@
 		)
 		(property "Description" "Power symbol creates a global label with name \"VBUS\""
-			(at 63.5 109.22 0)
+			(at 30.48 109.22 0)
 			(effects
 				(font
@@
 	(symbol
 		(lib_id "power:+3.3V")
-		(at 30.48 109.22 270)
-		(unit 1)
-		(exclude_from_sim no)
-		(in_bom yes)
-		(on_board yes)
-		(dnp no)
-		(fields_autoplaced yes)
+		(at 63.5 109.22 270)
+		(unit 1)
+		(exclude_from_sim no)
+		(in_bom yes)
+		(on_board yes)
+		(dnp no)
 		(property "Reference" "#PWR09"
-			(at 26.67 109.22 0)
+			(at 59.69 109.22 0)
 			(effects
 				(font
@@
 		)
 		(property "Value" "+3.3V"
-			(at 35.306 109.2199 90)
+			(at 66.548 109.22 90)
 			(effects
 				(font
@@
 		)
 		(property "Footprint" ""
-			(at 30.48 109.22 0)
+			(at 63.5 109.22 0)
 			(effects
 				(font
@@
 		)
 		(property "Datasheet" ""
-			(at 30.48 109.22 0)
+			(at 63.5 109.22 0)
 			(effects
 				(font
@@
 		)
 		(property "Description" "Power symbol creates a global label with name \"+3.3V\""
-			(at 30.48 109.22 0)
-			(effects
-				(font
+			(at 63.5 109.22 0)
+			(effects
+				(font
