File: STM32F401RE lite board.kicad_pcb (KiCad board)
At the start: 2 copper layers, 45 parts, among them J1 USB_B_Micro, J2 Conn_01x04_Pin, J3 Conn_01x05_Pin, J4 Conn_01x04_Pin, J5 Conn_01x05_Pin, J7 Conn_01x19_Pin, J8 Conn_01x22_Pin, SW1 SW_Push, SW2 SW_SPDT, U1 USBLC6-2SC6, U2 LD3985M33R_SOT23, U3 STM32F401RETx, Y1 8MHz(16pF)

Commit message: C9
Parts:
- removed R5, R6: 22Ω, Resistor_SMD:R_0402_1005Metric
- removed U1: USBLC6-2SC6, Package_TO_SOT_SMD:SOT-23-6
- moved C12 78.9 mm to (171.0, 47.3), turned to -90 degrees
- moved FB1 75.1 mm to (154.1, 51.6), turned to 90 degrees
- moved J7 74.8 mm to (174.2, 21.8), turned to -90 degrees
- moved C4 74.8 mm to (151.8, 39.3), turned to 90 degrees
- moved C1 74.6 mm to (155.9, 36.4)
- moved C7 69.9 mm to (151.7, 47.0), turned to 90 degrees
- moved J2 69.8 mm to (154.8, 30.0), turned to -90 degrees
- moved C13 69.5 mm to (90.7, 38.9)
- moved D1 69.3 mm to (90.6, 35.1)
- moved C10 68.0 mm to (148.9, 39.7), turned to -90 degrees
- moved C14 68.0 mm to (91.3, 42.0)
- moved Y1 66.8 mm to (144.9, 45.5), turned to 90 degrees
- moved C11 66.1 mm to (148.8, 43.8), turned to 90 degrees
- moved R4 65.2 mm to (169.8, 47.2), turned to 90 degrees
- moved R10 64.7 mm to (153.0, 34.5)
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Connections:
- J1 pad 2: Net-(J1-D-) -> /D -
- J1 pad 3: Net-(J1-D+) -> /D +

Commit message: C10
Parts:
- removed C1, C17, C2, C3, C4, C7: 100nF, Capacitor_SMD:C_0402_1005Metric
- removed C10, C11: 20pF, Capacitor_SMD:C_0402_1005Metric
- removed C12: 1nF, Capacitor_SMD:C_0402_1005Metric
- removed C13, C16: 1µF_X5R, Capacitor_SMD:C_0402_1005Metric
- removed C14, C9: 100nF, Capacitor_SMD:C_0603_1608Metric
- removed C15: 10nF_X7R, Capacitor_SMD:C_0402_1005Metric
- removed C18: 4.7µF, Capacitor_SMD:C_0805_2012Metric
- removed C5, C6: 10µF, Capacitor_SMD:C_0805_2012Metric
- removed C8: 1µF, Capacitor_SMD:C_0402_1005Metric
- removed D1: BAT60A, Diode_SMD:D_SOD-323
- removed D2, D3: LED, LED_SMD:LED_0603_1608Metric
- removed FB1: 100MHz120Ω, Inductor_SMD:L_0603_1608Metric
- removed J1: USB_B_Micro, Connector_USB:USB_Micro-B_Molex-105017-0001
- removed J2, J4: Conn_01x04_Pin, Connector_PinHeader_2.54mm:PinHeader_1x04_P2.54mm_Vertical
- removed J3, J5: Conn_01x05_Pin, Connector_PinHeader_2.54mm:PinHeader_1x05_P2.54mm_Vertical
- removed J7: Conn_01x19_Pin, Connector_PinHeader_2.54mm:PinHeader_1x19_P2.54mm_Vertical
- removed J8: Conn_01x22_Pin, Connector_PinHeader_2.54mm:PinHeader_1x22_P2.54mm_Vertical
- removed R1: 10KΩ, Resistor_SMD:R_0402_1005Metric
- removed R10, R9: 4.7KΩ, Resistor_SMD:R_0402_1005Metric
- removed R2, R3: 0Ω, Resistor_SMD:R_0402_1005Metric
- removed R4: 1MΩ, Resistor_SMD:R_0402_1005Metric
- removed R7, R8: 1KΩ, Resistor_SMD:R_0402_1005Metric
- removed SW1: SW_Push, Button_Switch_SMD:SW_Push_1TS009xxxx-xxxx-xxxx_6x6x5mm
- removed SW2: SW_SPDT, Button_Switch_SMD:SW_SPDT_CK_JS102011SAQN
- removed U2: LD3985M33R_SOT23, Package_TO_SOT_SMD:SOT-23-5
- removed U3: STM32F401RETx, Package_QFP:LQFP-64_10x10mm_P0.5mm
- removed Y1: 8MHz(16pF), Crystal:Crystal_HC49-4H_Vertical

Commit message: C11
Parts:
- added C1: 100nF, Capacitor_SMD:C_0402_1005Metric, F.Cu at (154.2, 88.2)
- added C10: 20pF, Capacitor_SMD:C_0402_1005Metric, F.Cu at (150.9, 93.0)
- added C11: 20pF, Capacitor_SMD:C_0402_1005Metric, F.Cu at (150.8, 95.1)
- added C12: 1nF, Capacitor_SMD:C_0402_1005Metric, F.Cu at (182.7, 98.2)
- added C13: 1µF_X5R, Capacitor_SMD:C_0402_1005Metric, F.Cu at (180.6, 85.0)
- added C14: 100nF, Capacitor_SMD:C_0603_1608Metric, F.Cu at (180.4, 83.6)
- added C15: 10nF_X7R, Capacitor_SMD:C_0402_1005Metric, F.Cu at (171.7, 83.6)
- added C16: 1µF_X5R, Capacitor_SMD:C_0402_1005Metric, F.Cu at (173.7, 87.2)
- added C17: 100nF, Capacitor_SMD:C_0402_1005Metric, F.Cu at (174.4, 88.5)
- added C18: 4.7µF, Capacitor_SMD:C_0805_2012Metric, F.Cu at (170.1, 95.3)
- added C2: 100nF, Capacitor_SMD:C_0402_1005Metric, F.Cu at (169.9, 91.5)
- added C3: 100nF, Capacitor_SMD:C_0402_1005Metric, F.Cu at (165.2, 83.4)
- added C4: 100nF, Capacitor_SMD:C_0402_1005Metric, F.Cu at (153.1, 93.2)
- added C5: 10µF, Capacitor_SMD:C_0805_2012Metric, F.Cu at (152.4, 90.6)
- added C6: 10µF, Capacitor_SMD:C_0805_2012Metric, F.Cu at (156.3, 98.3)
- added C7: 100nF, Capacitor_SMD:C_0402_1005Metric, F.Cu at (153.5, 97.9)
- added C8: 1µF, Capacitor_SMD:C_0402_1005Metric, F.Cu at (152.4, 96.6)
- added C9: 100nF, Capacitor_SMD:C_0603_1608Metric, F.Cu at (133.2, 91.6)
- added D1: BAT60A, Diode_SMD:D_SOD-323, F.Cu at (183.9, 85.0)
- added D2: LED, LED_SMD:LED_0603_1608Metric, F.Cu at (175.1, 92.4)
- added D3: LED, LED_SMD:LED_0603_1608Metric, F.Cu at (142.5, 90.7)
- added FB1: 100MHz120Ω, Inductor_SMD:L_0603_1608Metric, F.Cu at (155.0, 96.5)
- added J2: USB_C_Receptacle_USB2.0_16P, Connector_USB:USB_C_Receptacle_HRO_TYPE-C-31-M-12, F.Cu at (182.7, 91.5)
- added J3: Conn_01x05_Pin, Connector_PinHeader_2.54mm:PinHeader_1x05_P2.54mm_Vertical, F.Cu at (126.7, 86.5)
- added J6: Conn_01x24_Pin, Connector_PinHeader_2.54mm:PinHeader_1x24_P2.54mm_Vertical, F.Cu at (184.8, 79.4)
- added J9: Conn_01x24_Pin, Connector_PinHeader_2.54mm:PinHeader_1x24_P2.54mm_Vertical, F.Cu at (184.7, 103.2)
- added R1: 5.1KΩ, Resistor_SMD:R_0402_1005Metric, F.Cu at (175.4, 95.0)
- added R2: 10KΩ, Resistor_SMD:R_0402_1005Metric, F.Cu at (132.8, 90.0)
- added R3: 5.1KΩ, Resistor_SMD:R_0402_1005Metric, F.Cu at (176.0, 90.0)
- added R4: 1MΩ, Resistor_SMD:R_0402_1005Metric, F.Cu at (185.1, 98.2)
- added R5: 4.7KΩ, Resistor_SMD:R_0402_1005Metric, F.Cu at (156.1, 84.5)
- added R6: 4.7KΩ, Resistor_SMD:R_0402_1005Metric, F.Cu at (154.8, 86.0)
- added R7: 1KΩ, Resistor_SMD:R_0402_1005Metric, F.Cu at (175.4, 93.9)
- added R8: 1KΩ, Resistor_SMD:R_0402_1005Metric, F.Cu at (137.0, 90.6)
- added SW3: SW_SPST, Button_Switch_SMD:SW_SPST_TL3342, F.Cu at (136.0, 85.9)
- added SW4: SW_SPST, Button_Switch_SMD:SW_SPST_TL3342, F.Cu at (135.8, 95.6)
- added U2: LD3985M33R_SOT23, Package_TO_SOT_SMD:SOT-23-5, F.Cu at (174.8, 84.6)
- added U3: STM32F401RETx, Package_QFP:LQFP-64_10x10mm_P0.5mm, F.Cu at (161.7, 91.2)
- added Y1: 8MHz(16pF), Crystal:Crystal_HC49-4H_Vertical, F.Cu at (147.4, 93.3)
Routing:
- net /PA10/UART_RX: track 0.00 -> 28.1 mm
- net /PA9/UART_TX: track 0.00 -> 27.2 mm
- net /PA15: track 0.00 -> 22.0 mm
- net /D +: track 0.00 -> 17.7 mm
- net /D -: track 0.00 -> 17.2 mm
- net /OSC_IN: track 0.00 -> 12.8 mm
- net /OSC_OUT: track 0.00 -> 11.0 mm
Other:
- board text added: "UART"

Commit message: C12
Parts:
- moved R4 139.2 mm to (48.2, 72.9), turned to 0 degrees
- moved C12 131.2 mm to (53.9, 72.8), turned to 0 degrees
- moved R1 130.3 mm to (48.2, 66.9), turned to 0 degrees
- moved R3 129.3 mm to (48.2, 70.9)
- moved D1 128.3 mm to (55.9, 77.3)
- moved R7 128.1 mm to (48.2, 78.9), turned to 0 degrees
- moved C13 127.0 mm to (53.9, 74.8), turned to 0 degrees
- moved D2 124.4 mm to (51.7, 77.1), turned to 0 degrees
- moved C2 120.9 mm to (51.1, 68.9), turned to 0 degrees
- moved C17 118.9 mm to (56.8, 70.9)
- moved C16 118.3 mm to (56.8, 68.9)
- moved C15 116.1 mm to (56.8, 66.9), turned to 0 degrees
- moved C3 114.8 mm to (51.1, 70.9)
- moved C14 112.0 mm to (68.5, 80.6)
- moved U2 108.4 mm to (66.9, 74.1), turned to 0 degrees
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Connections:
- J6 pad 1: VBUS -> +3.3V
- J6 pad 10: /PB4 -> /PB15
- J6 pad 11: /PB5 -> /PB14
- J6 pad 12: /PB6/I2C_SCL -> /PB13
- J6 pad 13: /PB7/I2C_SDA -> /PB12
- J6 pad 14: /PB8 -> /PB10
- J6 pad 15: /PB9 -> /PB2
- J6 pad 16: /PC13 -> /PB1
- J6 pad 17: /PC14 -> /PB0
- J6 pad 18: /PC15 -> /PC5
- J6 pad 19: /PC0 -> /PC4
- J6 pad 2: /PA10/UART_RX -> GND
- J6 pad 20: /PC1 -> /PA7/SPI_MOSI
- J6 pad 21: /PC2 -> /PA6/SPI_MISO
- J6 pad 22: /PC3 -> /PA5/SPI_SCK
- J6 pad 23: /PA0 -> /PA4
- J6 pad 24: /PA1 -> /PA3
- J6 pad 3: /PA9/UART_TX -> /PA10/UART_RX
- J6 pad 4: /PA15 -> /PA9/UART_TX
- J6 pad 5: /PC10 -> /PA8
- J6 pad 6: /PC11 -> /PC9
- J6 pad 7: /PC12 -> /PC8
- J6 pad 8: /PD2 -> /PC7
- J6 pad 9: /PB3 -> /PC6
- J9 pad 1: +3.3V -> VBUS
- J9 pad 10: /PB14 -> /PB5
- J9 pad 11: /PB13 -> /PB6/I2C_SCL
- J9 pad 12: /PB12 -> /PB7/I2C_SDA
- J9 pad 13: /PB10 -> /PB8
- J9 pad 14: /PB2 -> /PB9
- J9 pad 15: /PB1 -> /PC13
- J9 pad 16: /PB0 -> /PC14
- J9 pad 17: /PC5 -> /PC15
- J9 pad 18: /PC4 -> /PC0
- J9 pad 19: /PA7/SPI_MOSI -> /PC1
- J9 pad 20: /PA6/SPI_MISO -> /PC2
- J9 pad 21: /PA5/SPI_SCK -> /PC3
- J9 pad 22: /PA4 -> /PA0
- J9 pad 23: /PA3 -> /PA1
- J9 pad 3: /PA8 -> /PA15
- J9 pad 4: /PC9 -> /PC10
- J9 pad 5: /PC8 -> /PC11
- J9 pad 6: /PC8 -> /PC12
- J9 pad 7: /PC7 -> /PD2
- J9 pad 8: /PC6 -> /PB3
- J9 pad 9: /PB15 -> /PB4
Routing:
- net /PA2: track 0.00 -> 52.7 mm, vias 0 -> 2
- net /PA1: track 0.00 -> 48.1 mm, vias 0 -> 2
- net /SWDIO: track 0.00 -> 44.8 mm, vias 0 -> 1
- net /PA0: track 0.00 -> 44.3 mm, vias 0 -> 2
- net /SWCLK: track 0.00 -> 43.8 mm, vias 0 -> 1
- net /NRST: track 0.00 -> 43.0 mm, vias 0 -> 2
- net /PC3: track 0.00 -> 37.1 mm
- net /PA4: track 0.00 -> 35.6 mm
- net /PA3: track 0.00 -> 35.5 mm
- net /PC2: track 0.00 -> 34.5 mm
- net /PA5/SPI_SCK: track 0.00 -> 33.6 mm
- net /PB0: track 0.00 -> 32.6 mm, vias 0 -> 1
- net /PC1: track 0.00 -> 31.8 mm
- net /PA6/SPI_MISO: track 0.00 -> 31.6 mm
- net /PA7/SPI_MOSI: track 0.00 -> 29.7 mm
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Other:
- board text removed: "UART"

Commit message: C13
Parts:
- moved R1 171.3 mm to (218.6, 84.1)
- moved R3 171.1 mm to (218.6, 86.2)
- moved R4 171.1 mm to (218.6, 88.1)
- moved R7 170.7 mm to (218.5, 90.3)
- moved D2 164.3 mm to (215.3, 91.6)
- moved D1 160.3 mm to (215.2, 94.6)
- moved C12 154.3 mm to (207.5, 88.3)
- moved C13 154.3 mm to (207.5, 90.3)
- moved C15 151.5 mm to (207.5, 82.3)
- moved C16 151.5 mm to (207.5, 84.3)
- moved C17 151.5 mm to (207.5, 86.3)
- moved C1 148.8 mm to (198.9, 84.1)
- moved C2 148.8 mm to (198.9, 86.0)
- moved C3 148.8 mm to (198.9, 88.0)
- moved C4 148.8 mm to (198.9, 90.0)
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Routing:
- net +3.3V: track 0.00 -> 122.1 mm, vias 0 -> 2
- net /PB13: track 0.00 -> 29.9 mm, vias 0 -> 1
- net /PB12: track 0.00 -> 20.7 mm, vias 0 -> 1
- net /PB14: track 0.00 -> 20.2 mm, vias 0 -> 1
- net /PB0: track 32.6 -> 12.7 mm
- net /SWDIO: track 44.8 -> 30.0 mm
- net /SWCLK: track 43.8 -> 28.9 mm
- net GND: track 0.00 -> 6.30 mm
- net Net-(U3-VCAP1): track 0.00 -> 4.27 mm
- net /BOOT0: track 5.35 -> 8.69 mm
- net +3.3VA: track 0.00 -> 2.79 mm
- net /PC7: track 13.9 -> 16.6 mm
- net /PB15: track 16.3 -> 18.6 mm
- net /PC6: track 15.0 -> 17.1 mm
- net /USER_LED_K: track 3.40 -> 2.17 mm
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Other:
- board text added: "BOOT"
- board text added: "NRST"

Commit message: C14
Parts:
- added REF**: KiCad-Logo2_6mm_SilkScreen, Symbol:KiCad-Logo2_6mm_SilkScreen, B.Cu at (125.7, 89.2)
- moved C5 53.6 mm to (146.4, 80.7), turned to 180 degrees
- moved R7 50.1 mm to (168.8, 84.2), turned to -90 degrees
- moved C2 49.4 mm to (149.6, 82.8), turned to 135 degrees
- moved D2 48.6 mm to (167.2, 84.8), turned to -90 degrees
- moved C1 48.4 mm to (150.5, 81.7), turned to 135 degrees
- moved R4 46.2 mm to (172.9, 81.1), turned to -90 degrees
- moved R3 44.8 mm to (174.1, 81.1), turned to -90 degrees
- moved R1 43.5 mm to (175.2, 81.1), turned to 90 degrees
- moved U2 42.0 mm to (170.5, 95.4), turned to 180 degrees
- moved C7 40.4 mm to (149.0, 93.7)
- moved C15 39.9 mm to (168.9, 92.5), turned to 90 degrees
- moved C16 39.5 mm to (168.3, 89.7)
- moved C17 39.5 mm to (168.3, 90.9)
- moved D1 38.2 mm to (177.0, 95.6), turned to 90 degrees
- moved C12 36.6 mm to (171.7, 81.1), turned to 90 degrees
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Connections:
- J6 pad 1: +3.3V -> VBUS
- J9 pad 1: VBUS -> +3.3V
Routing:
- net +3.3V: track 122.1 -> 209.1 mm, vias 2 -> 9
- net GND: track 6.30 -> 90.4 mm, vias 0 -> 18
- net /BOOT0: track 8.69 -> 44.2 mm, vias 0 -> 2
- net VBUS: track 0.00 -> 25.5 mm, vias 0 -> 3
- net +3.3VA: track 2.79 -> 27.2 mm, vias 0 -> 2
- net /PB0: track 12.7 -> 37.0 mm, vias 1 -> 2
- net Net-(J2-SHIELD): track 0.00 -> 20.6 mm
- net Net-(J2-CC1): track 0.00 -> 13.1 mm
- net Net-(D1-K): track 0.00 -> 9.48 mm
- net Net-(J2-CC2): track 0.00 -> 7.31 mm
- net /PWR_LED K: track 0.00 -> 2.29 mm
- net Net-(U2-BYP): track 0.00 -> 1.65 mm
- net /PA1: track 48.1 -> 49.8 mm
- net /PB13: track 29.9 -> 31.0 mm
- net /PB12: track 20.7 -> 19.7 mm
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- added copper zone on B.Cu, net GND
Other:
- board outline added: 62.8 x 41 mm
- board text added: "5V"
- board text added: "A10/RX"
- board text added: "A3"
- board text added: "A4"
- board text added: "A5/SCK"
- board text added: "A6/MISO"
- board text added: "A7/MOSI"
- board text added: "A9/TX"
- board text added: "B0"
- board text added: "B1"
- board text added: "B10"
- board text added: "B12"
- board text added: "B13"
- board text added: "B14"
- board text added: "B2"
- board text added: "B6/SCL"
- board text added: "B7/SDA"
- board text added: "C4"
- board text added: "C5"
- board text added: "Designed by, ANTONY"
- board text added: "GND"
- board text added: "I2C"
- board text added: "SPI"
- board text added: "UART"

Commit message: C15
Routing:
- net /PA2: track 52.9 -> 53.6 mm
Other:
- board text added: "3.3V"
- board text added: "A0"
- board text added: "A1"
- board text added: "A15"
- board text added: "A2"
- board text added: "A8"
- board text added: "B15"
- board text added: "B3"
- board text added: "B4"
- board text added: "B5"
- board text added: "B8"
- board text added: "B9"
- board text added: "C0"
- board text added: "C1"
- board text added: "C10"
- board text added: "C11"
- board text added: "C12"
- board text added: "C13"
- board text added: "C14"
- board text added: "C15"
- board text added: "C2"
- board text added: "C3"
- board text added: "C6"
- board text added: "C7"
- board text added: "C8"
- board text added: "C9"
- board text added: "CLK"
- board text added: "D2"
- board text added: "DIO"

Commit message: C16
Other:
- board text added: "RESET"
Changed lines of the file:
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@@
 		(tags "capacitor")
 		(property "Reference" "C5"
-			(at 2.65 0.06 0)
+			(at 2.95 -0.43 0)
 			(layer "F.SilkS")
 			(effects
@@
 		(tags "capacitor")
 		(property "Reference" "C1"
-			(at 1.449569 0.841457 0)
+			(at 1.244508 1.131371 0)
 			(layer "F.SilkS")
 			(effects
@@
 		(tags "capacitor")
 		(property "Reference" "C9"
-			(at -2.4 -0.04 180)
+			(at -2.55 -0.32 180)
 			(layer "F.SilkS")
 			(effects
@@
 	)
 	(gr_text "BOOT"
-		(at 116.38 81.1 270)
+		(at 116.52 81.13 270)
 		(layer "F.SilkS")
 		(effects
@@
 		)
 	)
-	(gr_text "NRST\n"
-		(at 116.46 89.35 270)
+	(gr_text "\nRESET\n"
+		(at 116.62 88.75 270)
 		(layer "F.SilkS")
 		(effects
